Commit message: adding panda gz simulation

File: aprs_ws/src/panda_description/urdf/panda.urdf (robot description, URDF)
Before this commit: robot panda, 12 links, 11 joints
Links:
- added link panda_hand_tcp
- added link world
- link panda_hand: mass None -> 0.14060765127978503; geometry collision mesh filename=package://panda_description/meshes/collision/hand.stl; visual mesh filename=package://panda_description/meshes/visual/hand.dae
- link panda_leftfinger: mass None -> 0.2238453537819424; geometry collision mesh filename=package://panda_description/meshes/collision/finger.stl; visual mesh filename=package://panda_description/meshes/visual/finger.dae
- link panda_link0: mass None -> 2.814271300104062; geometry collision mesh filename=package://panda_description/meshes/collision/link0.stl; visual mesh filename=package://panda_description/meshes/visual/link0.dae
- link panda_link1: mass None -> 2.6433170427227215; geometry collision mesh filename=package://panda_description/meshes/collision/link1.stl; visual mesh filename=package://panda_description/meshes/visual/link1.dae
- link panda_link2: mass None -> 2.6652755331661186; geometry collision mesh filename=package://panda_description/meshes/collision/link2.stl; visual mesh filename=package://panda_description/meshes/visual/link2.dae
- link panda_link3: mass None -> 2.3293714829045733; geometry collision mesh filename=package://panda_description/meshes/collision/link3.stl; visual mesh filename=package://panda_description/meshes/visual/link3.dae
- link panda_link4: mass None -> 2.3104763646281508; geometry collision mesh filename=package://panda_description/meshes/collision/link4.stl; visual mesh filename=package://panda_description/meshes/visual/link4.dae
- link panda_link5: mass None -> 2.6226426154892004; geometry collision mesh filename=package://panda_description/meshes/collision/link5.stl; visual mesh filename=package://panda_description/meshes/visual/link5.dae
- link panda_link6: mass None -> 1.5025804886626795; geometry collision mesh filename=package://panda_description/meshes/collision/link6.stl; visual mesh filename=package://panda_description/meshes/visual/link6.dae
- link panda_link7: mass None -> 0.5237668134788256; geometry collision mesh filename=package://panda_description/meshes/collision/link7.stl; visual mesh filename=package://panda_description/meshes/visual/link7.dae
- link panda_rightfinger: mass None -> 0.2238453537819424; geometry collision mesh filename=package://panda_description/meshes/collision/finger.stl; visual mesh filename=package://panda_description/meshes/visual/finger.dae
Joints:
- removed joint panda_hand_joint
- removed joint panda_joint8
- added joint panda_hand_tcp_virtual_joint: type fixed, parent panda_hand, child panda_hand_tcp, origin xyz=0 0 0.1034 rpy=0 0 0
- added joint panda_joint_base: type fixed, parent world, child panda_link0, origin xyz=0 0 0 rpy=0 0 0
- added joint panda_joint_wrist: type fixed, parent panda_link8, child panda_hand, origin xyz=0 0 0 rpy=0 0 0
- added joint panda_link8_virtual_joint: type fixed, parent panda_link7, child panda_link8, origin xyz=0 0 0.107 rpy=0 0 -0.7853981633974483
- joint panda_finger_joint1: limit lower=0.0 upper=0.04 effort=20 velocity=0.2 -> lower=0 upper=0.04 effort=20 velocity=0.2
- joint panda_finger_joint2: limit lower=0.0 upper=0.04 effort=20 velocity=0.2 -> lower=0 upper=0.04 effort=20 velocity=0.2; mimic joint=panda_finger_joint1 -> (none)
- joint panda_joint1: limit lower=-2.9671 upper=2.9671 effort=87 velocity=2.3925 -> lower=-2.897246558310587 upper=2.897246558310587 effort=87 velocity=2.6179938779914944
- joint panda_joint2: limit lower=-1.8326 upper=1.8326 effort=87 velocity=2.3925 -> lower=-1.7627825445142729 upper=1.7627825445142729 effort=87 velocity=2.6179938779914944; origin xyz=0 0 0 rpy=-1.57079632679 0 0 -> xyz=0 0 0 rpy=-1.5707963267948966 0 0
- joint panda_joint3: limit lower=-2.9671 upper=2.9671 effort=87 velocity=2.3925 -> lower=-2.897246558310587 upper=2.897246558310587 effort=87 velocity=2.6179938779914944; origin xyz=0 -0.316 0 rpy=1.57079632679 0 0 -> xyz=0 -0.316 0 rpy=1.5707963267948966 0 0
- joint panda_joint4: limit lower=-3.1416 upper=0.0873 effort=87 velocity=2.3925 -> lower=-3.07177948351002 upper=-0.06981317007977318 effort=87 velocity=2.6179938779914944; origin xyz=0.0825 0 0 rpy=1.57079632679 0 0 -> xyz=0.0825 0 0 rpy=1.5707963267948966 0 0
- joint panda_joint5: limit lower=-2.9671 upper=2.9671 effort=12 velocity=2.8710 -> lower=-2.897246558310587 upper=2.897246558310587 effort=12 velocity=3.141592653589793; origin xyz=-0.0825 0.384 0 rpy=-1.57079632679 0 0 -> xyz=-0.0825 0.384 0 rpy=-1.5707963267948966 0 0
- joint panda_joint6: limit lower=-0.0873 upper=3.8223 effort=12 velocity=2.8710 -> lower=-0.017453292519943295 upper=3.752457891787808 effort=12 velocity=3.141592653589793; origin xyz=0 0 0 rpy=1.57079632679 0 0 -> xyz=0 0 0 rpy=1.5707963267948966 0 0
- joint panda_joint7: limit lower=-2.9671 upper=2.9671 effort=12 velocity=2.8710 -> lower=-2.897246558310587 upper=2.897246558310587 effort=12 velocity=3.141592653589793; origin xyz=0.088 0 0 rpy=1.57079632679 0 0 -> xyz=0.088 0 0 rpy=1.5707963267948966 0 0
