Commit message: s2r not working test

File: aprs_ws/src/assets/robots/universal_robots/ur_description/urdf/ur.ros2_control.xacro (robot description, xacro)
@@ -3,9 +3,7 @@
   <xacro:macro name="ur_ros2_control" params="
     name
-    prefix
-    use_fake_hardware:=false fake_sensor_commands:=false
+    use_mock_hardware:=false mock_sensor_commands:=false
     sim_gazebo:=false
-    sim_gz:=false
-    real:=false
+    sim_ignition:=false
     headless_mode:=false
     initial_positions:=${dict(shoulder_pan_joint=0.0,shoulder_lift_joint=-1.57,elbow_joint=0.0,wrist_1_joint=-1.57,wrist_2_joint=0.0,wrist_3_joint=0.0)}
@@ -19,5 +17,9 @@
     script_sender_port:=50002
     reverse_ip:=0.0.0.0
-    script_command_port:=50004">
+    script_command_port:=50004
+    trajectory_port:=50003
+    non_blocking_read:=false
+    keep_alive_count:=2
+    ">
     <ros2_control name="${name}" type="system">
       <hardware>
@@ -25,13 +27,13 @@
           <plugin>gazebo_ros2_control/GazeboSystem</plugin>
         </xacro:if>
-        <xacro:if value="${sim_gz}">
+        <xacro:if value="${sim_ignition}">
           <plugin>gz_ros2_control/GazeboSimSystem</plugin>
         </xacro:if>
-        <xacro:if value="${use_fake_hardware}">
+        <xacro:if value="${use_mock_hardware}">
           <plugin>mock_components/GenericSystem</plugin>
-          <param name="fake_sensor_commands">${fake_sensor_commands}</param>
+          <param name="mock_sensor_commands">${mock_sensor_commands}</param>
           <param name="state_following_offset">0.0</param>
         </xacro:if>
-        <xacro:if value="${real}">
+        <xacro:unless value="${use_mock_hardware or sim_gazebo or sim_ignition}">
           <plugin>ur_robot_driver/URPositionHardwareInterface</plugin>
           <param name="robot_ip">${robot_ip}</param>
@@ -44,6 +46,7 @@
           <param name="reverse_ip">${reverse_ip}</param>
           <param name="script_command_port">${script_command_port}</param>
-          <param name="tf_prefix">"${tf_prefix}"</param>
-          <param name="non_blocking_read">0</param>
+          <param name="trajectory_port">${trajectory_port}</param>
+          <param name="tf_prefix">${tf_prefix}</param>
+          <param name="non_blocking_read">${non_blocking_read}</param>
           <param name="servoj_gain">2000</param>
           <param name="servoj_lookahead_time">0.03</param>
@@ -58,7 +61,8 @@
           <param name="tool_device_name">${tool_device_name}</param>
           <param name="tool_tcp_port">${tool_tcp_port}</param>
-        </xacro:if>
+          <param name="keep_alive_count">${keep_alive_count}</param>
+        </xacro:unless>
       </hardware>
-      <joint name="${prefix}shoulder_pan_joint">
+      <joint name="${tf_prefix}shoulder_pan_joint">
         <command_interface name="position">
           <param name="min">{-2*pi}</param>
@@ -70,11 +74,15 @@
         </command_interface>
         <state_interface name="position">
-          <!-- initial position for the FakeSystem and simulation -->
+          <!-- initial position for the mock system and simulation -->
           <param name="initial_value">${initial_positions['shoulder_pan_joint']}</param>
         </state_interface>
-        <state_interface name="velocity"/>
-        <state_interface name="effort"/>
-      </joint>
-      <joint name="${prefix}shoulder_lift_joint">
+        <state_interface name="velocity">
+          <param name="initial_value">0.0</param>
+        </state_interface>
+        <state_interface name="effort">
+          <param name="initial_value">0.0</param>
+        </state_interface>
+      </joint>
+      <joint name="${tf_prefix}shoulder_lift_joint">
         <command_interface name="position">
           <param name="min">{-2*pi}</param>
@@ -86,11 +94,15 @@
         </command_interface>
         <state_interface name="position">
-          <!-- initial position for the FakeSystem and simulation -->
+          <!-- initial position for the mock system and simulation -->
           <param name="initial_value">${initial_positions['shoulder_lift_joint']}</param>
         </state_interface>
-        <state_interface name="velocity"/>
-        <state_interface name="effort"/>
-      </joint>
-      <joint name="${prefix}elbow_joint">
+        <state_interface name="velocity">
+          <param name="initial_value">0.0</param>
+        </state_interface>
+        <state_interface name="effort">
+          <param name="initial_value">0.0</param>
+        </state_interface>
+      </joint>
+      <joint name="${tf_prefix}elbow_joint">
         <command_interface name="position">
           <param name="min">{-pi}</param>
@@ -102,11 +114,15 @@
         </command_interface>
         <state_interface name="position">
-          <!-- initial position for the FakeSystem and simulation -->
+          <!-- initial position for the mock system and simulation -->
           <param name="initial_value">${initial_positions['elbow_joint']}</param>
         </state_interface>
-        <state_interface name="velocity"/>
-        <state_interface name="effort"/>
-      </joint>
-      <joint name="${prefix}wrist_1_joint">
+        <state_interface name="velocity">
+          <param name="initial_value">0.0</param>
+        </state_interface>
+        <state_interface name="effort">
+          <param name="initial_value">0.0</param>
+        </state_interface>
+      </joint>
+      <joint name="${tf_prefix}wrist_1_joint">
         <command_interface name="position">
           <param name="min">{-2*pi}</param>
@@ -118,11 +134,15 @@
         </command_interface>
         <state_interface name="position">
-          <!-- initial position for the FakeSystem and simulation -->
+          <!-- initial position for the mock system and simulation -->
           <param name="initial_value">${initial_positions['wrist_1_joint']}</param>
         </state_interface>
-        <state_interface name="velocity"/>
-        <state_interface name="effort"/>
-      </joint>
-      <joint name="${prefix}wrist_2_joint">
+        <state_interface name="velocity">
+          <param name="initial_value">0.0</param>
+        </state_interface>
+        <state_interface name="effort">
+          <param name="initial_value">0.0</param>
+        </state_interface>
+      </joint>
+      <joint name="${tf_prefix}wrist_2_joint">
         <command_interface name="position">
           <param name="min">{-2*pi}</param>
@@ -134,11 +154,15 @@
         </command_interface>
         <state_interface name="position">
-          <!-- initial position for the FakeSystem and simulation -->
+          <!-- initial position for the mock system and simulation -->
           <param name="initial_value">${initial_positions['wrist_2_joint']}</param>
         </state_interface>
-        <state_interface name="velocity"/>
-        <state_interface name="effort"/>
-      </joint>
-      <joint name="${prefix}wrist_3_joint">
+        <state_interface name="velocity">
+          <param name="initial_value">0.0</param>
+        </state_interface>
+        <state_interface name="effort">
+          <param name="initial_value">0.0</param>
+        </state_interface>
+      </joint>
+      <joint name="${tf_prefix}wrist_3_joint">
         <command_interface name="position">
           <param name="min">{-2*pi}</param>
@@ -150,12 +174,16 @@
         </command_interface>
         <state_interface name="position">
-          <!-- initial position for the FakeSystem and simulation -->
+          <!-- initial position for the mock system and simulation -->
           <param name="initial_value">${initial_positions['wrist_3_joint']}</param>
         </state_interface>
-        <state_interface name="velocity"/>
-        <state_interface name="effort"/>
-      </joint>
-      <xacro:if value="${real}">
-        <sensor name="tcp_fts_sensor">
+        <state_interface name="velocity">
+          <param name="initial_value">0.0</param>
+        </state_interface>
+        <state_interface name="effort">
+          <param name="initial_value">0.0</param>
+        </state_interface>
+      </joint>
+      <xacro:unless value="${sim_gazebo or sim_ignition}">
+        <sensor name="${tf_prefix}tcp_fts_sensor">
           <state_interface name="force.x"/>
           <state_interface name="force.y"/>
@@ -165,6 +193,6 @@
           <state_interface name="torque.z"/>
         </sensor>
-        <!-- NOTE The following are joints used only for testing with fake hardware and will change in the future -->
-        <gpio name="speed_scaling">
+        <!-- NOTE The following are joints used only for testing with mock hardware and will change in the future -->
+        <gpio name="${tf_prefix}speed_scaling">
           <state_interface name="speed_scaling_factor"/>
           <param name="initial_speed_scaling_factor">1</param>
@@ -172,5 +200,5 @@
           <command_interface name="target_speed_fraction_async_success"/>
         </gpio>
-        <gpio name="gpio">
+        <gpio name="${tf_prefix}gpio">
           <command_interface name="standard_digital_output_cmd_0"/>
           <command_interface name="standard_digital_output_cmd_1"/>
@@ -266,5 +294,5 @@
           <state_interface name="program_running"/>
         </gpio>
-        <gpio name="payload">
+        <gpio name="${tf_prefix}payload">
           <command_interface name="mass"/>
           <command_interface name="cog.x"/>
@@ -273,16 +301,20 @@
           <command_interface name="payload_async_success"/>
         </gpio>
-        <gpio name="resend_robot_program">
+        <gpio name="${tf_prefix}resend_robot_program">
           <command_interface name="resend_robot_program_cmd"/>
           <command_interface name="resend_robot_program_async_success"/>
         </gpio>
-        <gpio name="zero_ftsensor">
+        <gpio name="${tf_prefix}hand_back_control">
+          <command_interface name="hand_back_control_cmd"/>
+          <command_interface name="hand_back_control_async_success"/>
+        </gpio>
+        <gpio name="${tf_prefix}zero_ftsensor">
           <command_interface name="zero_ftsensor_cmd"/>
           <command_interface name="zero_ftsensor_async_success"/>
         </gpio>
-        <gpio name="system_interface">
+        <gpio name="${tf_prefix}system_interface">
           <state_interface name="initialized"/>
         </gpio>
-      </xacro:if>
+      </xacro:unless>
     </ros2_control>
   </xacro:macro>

File: aprs_ws/src/assets/robots/universal_robots/ur_description/urdf/ur.urdf.xacro (robot description, xacro)
@@ -9,5 +9,5 @@
    <xacro:arg name="ur_type" default="ur5x"/>
    <!-- parameters -->
-   <xacro:arg name="prefix" default="" />
+   <xacro:arg name="tf_prefix" default="" />
    <xacro:arg name="joint_limit_params" default="$(find ur_description)/config/$(arg ur_type)/joint_limits.yaml"/>
    <xacro:arg name="kinematics_params" default="$(find ur_description)/config/$(arg ur_type)/default_kinematics.yaml"/>
@@ -37,11 +37,10 @@
    <xacro:arg name="tool_tcp_port" default="54321" />
      <!-- Simulation parameters -->
-   <xacro:arg name="use_fake_hardware" default="false" />
-   <xacro:arg name="fake_sensor_commands" default="false" />
+   <xacro:arg name="use_mock_hardware" default="false" />
+   <xacro:arg name="mock_sensor_commands" default="false" />
    <xacro:arg name="sim_gazebo" default="false" />
-   <xacro:arg name="sim_gz" default="false" />
-   <xacro:arg name="real" default="false" />
+   <xacro:arg name="sim_ignition" default="false" />
    <xacro:arg name="simulation_controllers" default="" />
-   <!-- initial position for simulations (Fake Hardware, Gazebo, Ignition) -->
+   <!-- initial position for simulations (Mock Hardware, Gazebo, Ignition) -->
    <xacro:arg name="initial_positions_file" default="$(find ur_description)/config/initial_positions.yaml"/>
    <!-- convert to property to use substitution in function -->
@@ -52,5 +51,5 @@
    <xacro:ur_robot
      name="$(arg name)"
-     prefix="$(arg prefix)"
+     tf_prefix="$(arg tf_prefix)"
      parent="world"
      joint_limits_parameters_file="$(arg joint_limit_params)"
@@ -62,9 +61,8 @@
      safety_pos_margin="$(arg safety_pos_margin)"
      safety_k_position="$(arg safety_k_position)"
-     use_fake_hardware="$(arg use_fake_hardware)"
-     fake_sensor_commands="$(arg fake_sensor_commands)"
+     use_mock_hardware="$(arg use_mock_hardware)"
+     mock_sensor_commands="$(arg mock_sensor_commands)"
      sim_gazebo="$(arg sim_gazebo)"
-     sim_gz="$(arg sim_gz)"
-     real="$(arg real)"
+     sim_ignition="$(arg sim_ignition)"
      headless_mode="$(arg headless_mode)"
      initial_positions="${xacro.load_yaml(initial_positions_file)}"
@@ -97,5 +95,5 @@
     </gazebo>
   </xacro:if>
-  <xacro:if value="$(arg sim_gz)">
+  <xacro:if value="$(arg sim_ignition)">
     <!-- Gazebo plugins -->
     <gazebo reference="world">
@@ -104,7 +102,28 @@
       <plugin filename="libgz_ros2_control-system.so" name="gz_ros2_control::GazeboSimROS2ControlPlugin">
         <parameters>$(arg simulation_controllers)</parameters>
-        <controller_manager_node_name>$(arg prefix)controller_manager</controller_manager_node_name>
+        <controller_manager_node_name>$(arg tf_prefix)controller_manager</controller_manager_node_name>
       </plugin>
     </gazebo>
   </xacro:if>
+  <gazebo reference="shoulder_link">
+      <selfCollide>true</selfCollide>
+  </gazebo>
+  <gazebo reference="upper_arm_link">
+    <selfCollide>true</selfCollide>
+  </gazebo>
+  <gazebo reference="forearm_link">
+    <selfCollide>true</selfCollide>
+  </gazebo>
+  <gazebo reference="wrist_1_link">
+    <selfCollide>true</selfCollide>
+  </gazebo>
+  <gazebo reference="wrist_3_link">
+    <selfCollide>true</selfCollide>
+  </gazebo>
+  <gazebo reference="wrist_2_link">
+    <selfCollide>true</selfCollide>
+  </gazebo>
+  <gazebo reference="ee_link">
+    <selfCollide>true</selfCollide>
+  </gazebo>
 </robot>
