Commit message: gripper simulation

File: aprs_ws/src/assets/robots/ur5e/ur_description/urdf/ur.urdf.xacro (robot description, xacro)
@@ -5,7 +5,8 @@
    <!-- import main macro -->
    <xacro:include filename="$(find ur_description)/urdf/ur_macro.xacro"/>
+   <!-- <xacro:include filename="$(find vaccum_description)/urdf/vaccum.urdf.xacro"/> -->
    <!-- possible 'ur_type' values: ur3, ur3e, ur5, ur5e, ur10, ur10e, ur16e -->
    <!-- the default value should raise an error in case this was called without defining the type -->
-   <xacro:arg name="ur_type" default="ur5x"/>
+   <xacro:arg name="ur_type" default="ur5e"/>
    <!-- parameters -->
    <xacro:arg name="prefix" default="" />
@@ -87,4 +88,7 @@
      <origin xyz="0 0 0" rpy="0 0 0" />          <!-- position robot in the world -->
    </xacro:ur_robot>
+   <!-- <xacro:vaccum_gripper prefix="" parent="tool0" >
+     <origin xyz="0.0 0 0.0" rpy="0 0 0"/>
+   </xacro:vaccum_gripper> -->
    <xacro:if value="$(arg sim_gazebo)">
     <!-- Gazebo plugins -->

File: aprs_ws/src/assets/robots/ur5e/ur_description/urdf/ur_macro.xacro (robot description, xacro)
@@ -337,10 +337,12 @@
       <dynamics damping="0" friction="0"/>
     </joint>
-    <link name="${prefix}ft_frame"/>
-    <joint name="${prefix}wrist_3_link-ft_frame" type="fixed">
-      <parent link="${prefix}wrist_3_link"/>
-      <child link="${prefix}ft_frame"/>
-      <origin xyz="0 0 0" rpy="${pi} 0 0"/>
-    </joint>
+    <xacro:include filename="$(find vaccum_description)/urdf/vaccum.urdf.xacro"/>
+    <xacro:vaccum_gripper prefix="" parent="wrist_3_link" >
+     <origin xyz="0.0 0.0 -0.02" rpy="${pi/2.0} 0 ${pi}"/>
+    </xacro:vaccum_gripper>
+    <!-- <xacro:include filename="$(find camera_mount)/urdf/camera_mount.urdf.xacro"/>
+    <xacro:camera_mount prefix="" parent="vaccum_e_link" >
+      <origin xyz="0.0 0.0 -0.02" rpy="${pi/2.0} 0 ${pi}"/>
+    </xacro:camera_mount> -->
     <!-- ROS-Industrial 'base' frame - base_link to UR 'Base' Coordinates transform -->
     <link name="${prefix}base"/>

File: aprs_ws/src/ur/urdf/vaccum.urdf.xacro (robot description, xacro)
@@ -11,5 +11,5 @@
         <origin rpy="0 0 0" xyz="0 0 0"/>
         <geometry>
-          <mesh filename="file://$(find ur)/meshes/vaccum_gripper.stl" scale="0.0001 0.0001 0.0001"/>
+          <mesh filename="file://$(find vaccum_description)/meshes/VaccumGripper.stl" scale="0.0001 0.0001 0.0001"/>
         </geometry>
         <material name="Dark">
@@ -20,5 +20,5 @@
         <origin rpy="0 0 0" xyz="0 0 0"/>
         <geometry>
-          <mesh filename="file://$(find ur)/meshes/vaccum_gripper.stl" scale="0.0001 0.0001 0.0001"/>
+          <mesh filename="file://$(find vaccum_description)/meshes/VaccumGripper.stl" scale="0.0001 0.0001 0.0001"/>
         </geometry>
       </collision>
