Commit message: panda gripper not woking

File: aprs_ws/src/assets/robots/panda_robot/panda_description/urdf/panda_arm.xacro (robot description, xacro)
@@ -82,5 +82,5 @@
   <xacro:property name="joint6_type" value="revolute"/>
   <xacro:property name="joint6_origin_xyz" value="0 0 0"/>
-  <xacro:property name="joint6_origin_rpy" value="${pi/2} 0 0"/>
+  <xacro:property name="joint6_origin_rpy" value="${-pi/2} 0 0"/>
   <xacro:property name="joint6_axis_xyz" value="0 0 1"/>
   <xacro:property name="joint6_lower_limit" value="${-1/180*pi}"/>
@@ -125,5 +125,5 @@
     ros2_control:=true
     ros2_control_plugin:=ign
-    ros2_control_command_interface:=effort
+    ros2_control_command_interface:=position
     gazebo_preserve_fixed_joint:=false
   ">

File: aprs_ws/src/assets/robots/panda_robot/panda_description/urdf/panda_gripper.xacro (robot description, xacro)
@@ -57,5 +57,5 @@
     collision:=true
     ros2_control:=true
-    ros2_control_plugin:=fakez
+    ros2_control_plugin:=ign
     ros2_control_command_interface:=effort
     gazebo_preserve_fixed_joint:=false

File: aprs_ws/src/assets/robots/panda_robot/panda_moveit_config/srdf/panda_gripper.xacro (robot description, xacro)
@@ -6,5 +6,5 @@
   <!--       -->
   <xacro:macro name="panda_gripper" params="
-    prefix:=franka_
+    prefix:=panda_
   ">
     <group name="gripper">
