Commit message: franka simulation with garden working

File: aprs_ws/src/assets/robots/panda_robot/panda_description/urdf/panda.urdf.xacro (robot description, xacro)
@@ -1,226 +1,99 @@
-<?xml version="1.0" ?>
-<!-- =================================================================================== -->
-<!-- |    This document was autogenerated by xacro from /opt/ros/kinetic/share/moveit_resources/panda_description/urdf/panda.urdf | -->
-<!-- |    EDITING THIS FILE BY HAND IS NOT RECOMMENDED                                 | -->
-<!-- =================================================================================== -->
-<robot xmlns:xacro="http://www.ros.org/wiki/xacro">
-<xacro:macro name="panda_robot">
-    <link name="panda_link0">
-        <visual>
-            <geometry>
-                <mesh filename="package://moveit_resources_panda_description/meshes/visual/link0.dae" />
-            </geometry>
-        </visual>
-        <collision>
-            <geometry>
-                <mesh filename="package://moveit_resources_panda_description/meshes/collision/link0.stl" />
-            </geometry>
-        </collision>
-    </link>
-    <link name="panda_link1">
-        <visual>
-            <geometry>
-                <mesh filename="package://moveit_resources_panda_description/meshes/visual/link1.dae" />
-            </geometry>
-        </visual>
-        <collision>
-            <geometry>
-                <mesh filename="package://moveit_resources_panda_description/meshes/collision/link1.stl" />
-            </geometry>
-        </collision>
-    </link>
-    <joint name="panda_joint1" type="revolute">
-        <safety_controller k_position="100.0" k_velocity="40.0" soft_lower_limit="-2.8973" soft_upper_limit="2.8973" />
-        <origin rpy="0 0 0" xyz="0 0 0.333" />
-        <parent link="panda_link0" />
-        <child link="panda_link1" />
-        <axis xyz="0 0 1" />
-        <limit effort="87" lower="-2.9671" upper="2.9671" velocity="2.3925" />
-    </joint>
-    <link name="panda_link2">
-        <visual>
-            <geometry>
-                <mesh filename="package://moveit_resources_panda_description/meshes/visual/link2.dae" />
-            </geometry>
-        </visual>
-        <collision>
-            <geometry>
-                <mesh filename="package://moveit_resources_panda_description/meshes/collision/link2.stl" />
-            </geometry>
-        </collision>
-    </link>
-    <joint name="panda_joint2" type="revolute">
-        <safety_controller k_position="100.0" k_velocity="40.0" soft_lower_limit="-1.7628" soft_upper_limit="1.7628" />
-        <origin rpy="-1.57079632679 0 0" xyz="0 0 0" />
-        <parent link="panda_link1" />
-        <child link="panda_link2" />
-        <axis xyz="0 0 1" />
-        <limit effort="87" lower="-1.8326" upper="1.8326" velocity="2.3925" />
-    </joint>
-    <link name="panda_link3">
-        <visual>
-            <geometry>
-                <mesh filename="package://moveit_resources_panda_description/meshes/visual/link3.dae" />
-            </geometry>
-        </visual>
-        <collision>
-            <geometry>
-                <mesh filename="package://moveit_resources_panda_description/meshes/collision/link3.stl" />
-            </geometry>
-        </collision>
-    </link>
-    <joint name="panda_joint3" type="revolute">
-        <safety_controller k_position="100.0" k_velocity="40.0" soft_lower_limit="-2.8973" soft_upper_limit="2.8973" />
-        <origin rpy="1.57079632679 0 0" xyz="0 -0.316 0" />
-        <parent link="panda_link2" />
-        <child link="panda_link3" />
-        <axis xyz="0 0 1" />
-        <limit effort="87" lower="-2.9671" upper="2.9671" velocity="2.3925" />
-    </joint>
-    <link name="panda_link4">
-        <visual>
-            <geometry>
-                <mesh filename="package://moveit_resources_panda_description/meshes/visual/link4.dae" />
-            </geometry>
-        </visual>
-        <collision>
-            <geometry>
-                <mesh filename="package://moveit_resources_panda_description/meshes/collision/link4.stl" />
-            </geometry>
-        </collision>
-    </link>
-    <joint name="panda_joint4" type="revolute">
-        <safety_controller k_position="100.0" k_velocity="40.0" soft_lower_limit="-3.0718" soft_upper_limit="0.0175" />
-        <origin rpy="1.57079632679 0 0" xyz="0.0825 0 0" />
-        <parent link="panda_link3" />
-        <child link="panda_link4" />
-        <axis xyz="0 0 1" />
-        <limit effort="87" lower="-3.1416" upper="0.0873" velocity="2.3925" />
-    </joint>
-    <link name="panda_link5">
-        <visual>
-            <geometry>
-                <mesh filename="package://moveit_resources_panda_description/meshes/visual/link5.dae" />
-            </geometry>
-        </visual>
-        <collision>
-            <geometry>
-                <mesh filename="package://moveit_resources_panda_description/meshes/collision/link5.stl" />
-            </geometry>
-        </collision>
-    </link>
-    <joint name="panda_joint5" type="revolute">
-        <safety_controller k_position="100.0" k_velocity="40.0" soft_lower_limit="-2.8973" soft_upper_limit="2.8973" />
-        <origin rpy="-1.57079632679 0 0" xyz="-0.0825 0.384 0" />
-        <parent link="panda_link4" />
-        <child link="panda_link5" />
-        <axis xyz="0 0 1" />
-        <limit effort="12" lower="-2.9671" upper="2.9671" velocity="2.8710" />
-    </joint>
-    <link name="panda_link6">
-        <visual>
-            <geometry>
-                <mesh filename="package://moveit_resources_panda_description/meshes/visual/link6.dae" />
-            </geometry>
-        </visual>
-        <collision>
-            <geometry>
-                <mesh filename="package://moveit_resources_panda_description/meshes/collision/link6.stl" />
-            </geometry>
-        </collision>
-    </link>
-    <joint name="panda_joint6" type="revolute">
-        <safety_controller k_position="100.0" k_velocity="40.0" soft_lower_limit="-0.0175" soft_upper_limit="3.7525" />
-        <origin rpy="1.57079632679 0 0" xyz="0 0 0" />
-        <parent link="panda_link5" />
-        <child link="panda_link6" />
-        <axis xyz="0 0 1" />
-        <limit effort="12" lower="-0.0873" upper="3.8223" velocity="2.8710" />
-    </joint>
-    <link name="panda_link7">
-        <visual>
-            <geometry>
-                <mesh filename="package://moveit_resources_panda_description/meshes/visual/link7.dae" />
-            </geometry>
-        </visual>
-        <collision>
-            <geometry>
-                <mesh filename="package://moveit_resources_panda_description/meshes/collision/link7.stl" />
-            </geometry>
-        </collision>
-    </link>
-    <joint name="panda_joint7" type="revolute">
-        <safety_controller k_position="100.0" k_velocity="40.0" soft_lower_limit="-2.8973" soft_upper_limit="2.8973" />
-        <origin rpy="1.57079632679 0 0" xyz="0.088 0 0" />
-        <parent link="panda_link6" />
-        <child link="panda_link7" />
-        <axis xyz="0 0 1" />
-        <limit effort="12" lower="-2.9671" upper="2.9671" velocity="2.8710" />
-    </joint>
-    <link name="panda_link8" />
-    <joint name="panda_joint8" type="fixed">
-        <origin rpy="0 0 0" xyz="0 0 0.107" />
-        <parent link="panda_link7" />
-        <child link="panda_link8" />
-        <axis xyz="0 0 0" />
-    </joint>
-    <joint name="panda_hand_joint" type="fixed">
-        <parent link="panda_link8" />
-        <child link="panda_hand" />
-        <origin rpy="0 0 -0.785398163397" xyz="0 0 0" />
-    </joint>
-    <link name="panda_hand">
-        <visual>
-            <geometry>
-                <mesh filename="package://moveit_resources_panda_description/meshes/visual/hand.dae" />
-            </geometry>
-        </visual>
-        <collision>
-            <geometry>
-                <mesh filename="package://moveit_resources_panda_description/meshes/collision/hand.stl" />
-            </geometry>
-        </collision>
-    </link>
-    <link name="panda_leftfinger">
-        <visual>
-            <geometry>
-                <mesh filename="package://moveit_resources_panda_description/meshes/visual/finger.dae" />
-            </geometry>
-        </visual>
-        <collision>
-            <geometry>
-                <mesh filename="package://moveit_resources_panda_description/meshes/collision/finger.stl" />
-            </geometry>
-        </collision>
-    </link>
-    <link name="panda_rightfinger">
-        <visual>
-            <origin rpy="0 0 3.14159265359" xyz="0 0 0" />
-            <geometry>
-                <mesh filename="package://moveit_resources_panda_description/meshes/visual/finger.dae" />
-            </geometry>
-        </visual>
-        <collision>
-            <origin rpy="0 0 3.14159265359" xyz="0 0 0" />
-            <geometry>
-                <mesh filename="package://moveit_resources_panda_description/meshes/collision/finger.stl" />
-            </geometry>
-        </collision>
-    </link>
-    <joint name="panda_finger_joint1" type="prismatic">
-        <parent link="panda_hand" />
-        <child link="panda_leftfinger" />
-        <origin rpy="0 0 0" xyz="0 0 0.0584" />
-        <axis xyz="0 1 0" />
-        <limit effort="20" lower="0.0" upper="0.04" velocity="0.2" />
-    </joint>
-    <joint name="panda_finger_joint2" type="prismatic">
-        <parent link="panda_hand" />
-        <child link="panda_rightfinger" />
-        <origin rpy="0 0 0" xyz="0 0 0.0584" />
-        <axis xyz="0 -1 0" />
-        <limit effort="20" lower="0.0" upper="0.04" velocity="0.2" />
-        <mimic joint="panda_finger_joint1" />
-    </joint>
-</xacro:macro>
+<?xml version="1.0"?>
+<!-- URDF for Franka Emika Panda -->
+<robot xmlns:xacro="http://wiki.ros.org/xacro" name="$(arg name)">
+  <!--                   -->
+  <!-- Imported elements -->
+  <!--                   -->
+  <xacro:include filename="$(find panda_description)/urdf/panda_arm.xacro"/>
+  <xacro:include filename="$(find panda_description)/urdf/panda_gripper.xacro"/>
+  <xacro:include filename="$(find panda_description)/urdf/panda_utils.xacro"/>
+  <xacro:include filename="$(find panda_description)/urdf/panda.gazebo"/>
+  <!--            -->
+  <!-- Parameters -->
+  <!--            -->
+  <!-- Name of the robot (mandatory) -->
+  <xacro:arg name="name" default="panda"/>
+  <!-- Prefix for all entities -->
+  <xacro:arg name="prefix" default="$(arg name)_"/>
+  <!-- Flag to enable default gripper -->
+  <xacro:arg name="gripper" default="true" />
+  <!-- Flag to enable collision geometry for manipulator's arm -->
+  <xacro:arg name="collision_arm" default="true"/>
+  <!-- Flag to enable collision geometry for manipulator's gripper (hand and fingers) -->
+  <xacro:arg name="collision_gripper" default="true"/>
+  <!-- Flag to enable safety limits controllers on manipulator joints -->
+  <xacro:arg name="safety_limits" default="false"/>
+  <!-- Lower and upper margin for position limits of all safety controllers -->
+  <xacro:arg name="safety_position_margin" default="0.17453293"/>
+  <!-- Parametric k-position factor of all safety controllers -->
+  <xacro:arg name="safety_k_position" default="100.0"/>
+  <!-- Parametric k-velocity factor of all safety controllers -->
+  <xacro:arg name="safety_k_velocity" default="40.0"/>
+  <!-- Flag to enable ros2 controllers for manipulator -->
+  <xacro:arg name="ros2_control" default="true"/>
+  <!-- The ros2_control plugin that should be loaded for the manipulator ('fake', 'ign', 'real' or custom) -->
+  <xacro:arg name="ros2_control_plugin" default="ign"/>
+  <!-- The output control command interface provided by ros2_control ('position', 'velocity', 'effort' or certain combinations 'position,velocity') -->
+  <xacro:arg name="ros2_control_command_interface" default="position"/>
+  <!-- The filepath to parameters of ROS 2 controllers -->
+  <xacro:arg name="ros2_controller_parameters" default="$(find franka_gz)/config/franka_controller.yaml"/>
+  <!-- Flag to preserve fixed joints and prevent lumping when generating SDF for Gazebo -->
+  <xacro:arg name="gazebo_preserve_fixed_joint" default="false"/>
+  <!--            -->
+  <!-- Properties -->
+  <!--            -->
+  <!-- Prefixes -->
+  <xacro:property name="prefix_arm" value="$(arg prefix)"/>
+  <xacro:property name="prefix_gripper" value="$(arg prefix)"/>
+  <!-- Origin of arm in the world -->
+  <xacro:property name="world_name" value="world"/>
+  <xacro:property name="origin_xyz" value="0 0 0"/>
+  <xacro:property name="origin_rpy" value="0 0 0"/>
+  <!-- Offset of gripper with respect to wrist flange -->
+  <xacro:property name="gripper_offset_xyz" value="0 0 0"/>
+  <xacro:property name="gripper_offset_rpy" value="0 0 0"/>
+  <!--       -->
+  <!-- Robot -->
+  <!--       -->
+  <!-- Dummy world link that the robot is fixed to -->
+  <xacro:panda_dummy_link
+    link_name="${world_name}"
+    gazebo_preserve_fixed_joint="$(arg gazebo_preserve_fixed_joint)"
+  />
+  <!-- Arm -->
+  <xacro:panda_arm
+    base_parent="world"
+    prefix="${prefix_arm}"
+    origin_xyz="${origin_xyz}"
+    origin_rpy="${origin_rpy}"
+    collision="$(arg collision_arm)"
+    safety_limits="$(arg safety_limits)"
+    safety_position_margin="$(arg safety_position_margin)"
+    safety_k_position="$(arg safety_k_position)"
+    safety_k_velocity="$(arg safety_k_velocity)"
+    ros2_control="$(arg ros2_control)"
+    ros2_control_plugin="$(arg ros2_control_plugin)"
+    ros2_control_command_interface="$(arg ros2_control_command_interface)"
+    gazebo_preserve_fixed_joint="$(arg gazebo_preserve_fixed_joint)"
+  />
+  <!-- Gripper -->
+  <xacro:if value="$(arg gripper)">
+    <xacro:panda_gripper
+      wrist_flange="${prefix_arm}${wrist_flange_name}"
+      prefix="${prefix_gripper}"
+      origin_xyz="${gripper_offset_xyz}"
+      origin_rpy="${gripper_offset_rpy}"
+      collision="$(arg collision_gripper)"
+      ros2_control="$(arg ros2_control)"
+      ros2_control_plugin="$(arg ros2_control_plugin)"
+      ros2_control_command_interface="$(arg ros2_control_command_interface)"
+      gazebo_preserve_fixed_joint="$(arg gazebo_preserve_fixed_joint)"
+    />
+  </xacro:if>
+  <!-- Gazebo - ROS 2 control (Ignition) -->
+  <xacro:if value="$(arg ros2_control)">
+    <xacro:if value="${'ign' in '$(arg ros2_control_plugin)'}">
+      <xacro:ign_ros2_control controller_parameters="$(arg ros2_controller_parameters)"/>
+    </xacro:if>
+  </xacro:if>
 </robot>

Commit message: aprs lab and multi arm in world sdf

File: aprs_ws/src/assets/robots/panda_robot/panda_description/urdf/panda.urdf.xacro (robot description, xacro)
@@ -48,5 +48,5 @@
   <!-- Origin of arm in the world -->
   <xacro:property name="world_name" value="world"/>
-  <xacro:property name="origin_xyz" value="0 0 0"/>
+  <xacro:property name="origin_xyz" value="2 0 0"/>
   <xacro:property name="origin_rpy" value="0 0 0"/>
   <!-- Offset of gripper with respect to wrist flange -->
