Commit message: humble ur with gripper simulation

File: aprs_ws/src/assets/end_effectors/VacuumGripper/urdf/vaccum.urdf.xacro (robot description, xacro)
@@ -4,5 +4,5 @@
     <link name="${prefix}vaccum_e_link">
       <visual>
-        <origin rpy="0 0 0" xyz="0 0 0"/>
+        <origin rpy="0 -1.5708 0" xyz="0 0 0"/>
         <geometry>
           <mesh filename="file://$(find vaccum_description)/meshes/VacuumGripper.stl" scale="1 1 1"/>
