Commit message: camera and vaccum urdf to ur description

File: aprs_ws/src/assets/robots/ur5e/Universal_Robots_ROS2_Description/urdf/ur.urdf.xacro (robot description, xacro)
@@ -6,4 +6,5 @@
    <xacro:include filename="$(find ur_description)/urdf/ur_macro.xacro"/>
    <xacro:include filename="$(find vaccum_description)/urdf/vaccum.urdf.xacro"/>
+   <xacro:include filename="$(find camera_mount)/urdf/camera_mount.urdf.xacro"/>
    <!-- possible 'ur_type' values: ur3, ur3e, ur5, ur5e, ur10, ur10e, ur16e, ur20 -->
    <!-- the default value should raise an error in case this was called without defining the type -->
@@ -89,4 +90,7 @@
      <origin xyz="0.0 0 -0.02" rpy="${pi/2.0} 0 ${pi}"/>
    </xacro:vaccum_gripper>
+   <xacro:camera_mount prefix="" parent="vaccum_e_link" >
+     <origin xyz="0.0 0 -0.02" rpy="${pi/2.0} 0 ${pi}"/>
+   </xacro:camera_mount>
    <xacro:if value="$(arg sim_gazebo)">
     <!-- Gazebo plugins -->

File: aprs_ws/src/assets/sensors/camera_mount/urdf/camera_mount.urdf.xacro (robot description, xacro)
@@ -21,6 +21,6 @@
     </link>
     <joint name="camera_mount_to_flange_joint" type="fixed">
-      <origin xyz="0.03 0 .045" rpy="0 0 0"/>
-      <parent link="vaccum_e_link"/>
+      <origin xyz="0 0 0" rpy="${pi/2.0} ${pi/2.0} ${pi}"/>
+      <parent link="flange"/>
       <child link="camera_mount" />
     </joint>
@@ -31,11 +31,11 @@
     </joint> -->
     <!-- Run camera macro -->
-    <!-- <xacro:sensor_d435
+    <xacro:sensor_d435
       parent="camera_mount"
       use_nominal_extrinsics="false"
       add_plug="false"
       use_mesh="true">
-      <origin xyz="0 0 0" rpy="0 0 0"/>
-    </xacro:sensor_d435> -->
+      <origin xyz="0 0 0" rpy="${pi/2.0} 0 ${-pi/2.0}"/>
+    </xacro:sensor_d435>
   </xacro:macro>
 </robot>
