Commit message: robots simulated, controllers not working

File: aprs_ws/src/assets/aprs_lab/urdf/aprs.urdf.xacro (robot description, xacro)
@@ -2,5 +2,5 @@
 <robot xmlns:xacro="http://www.ros.org/wiki/xacro" name="aprs_robots">
     <!-- Root link -->
-  <link name="world"/>
+  <!-- <link name="world"/> -->
   <!-- Material for RVIZ -->
   <material name="Grey">
@@ -11,4 +11,6 @@
   <!-- ur Robot -->
   <xacro:aprs_ur_robot/>
+  <xacro:include filename="$(find aprs_lab)/urdf/franka_robot_macro.xacro"/>
+  <xacro:aprs_franka_robot/>
   <gazebo
     reference="world">
@@ -22,5 +24,5 @@
       <plugin filename="libign_ros2_control-system.so" name="ign_ros2_control::IgnitionROS2ControlPlugin">
         <parameters>$(arg controllers)</parameters>
-        <!-- <controller_manager_node_name>controller_manager</controller_manager_node_name> -->
+         <controller_manager_node_name>controller_manager</controller_manager_node_name>
       </plugin>
     </gazebo>
