Commit message: gear launch

File: aprs_ws/src/assets/sensors/camera_mount/urdf/camera_mount.urdf.xacro (robot description, xacro)
@@ -22,10 +22,35 @@
     <!-- Camera Link -->
       <link name ="robot_camera_link">
-        <!-- <visual>
-          <origin xyz="0 0 0" rpy="0 0 0"/>
-          <geometry>
-            <mesh filename="file://$(find camera_mount)/meshes/camera.stl" scale="1 1 1"/>
-          </geometry>
-        </visual> -->
+        <sensor name="depth_camera" type="camera">
+          <always_on>true</always_on>
+          <visualize>false</visualize>
+          <update_rate>5</update_rate>
+          <camera name="camera">
+            <horizontal_fov>1.02974</horizontal_fov>
+            <image>
+              <width>640</width>
+              <height>480</height>
+              <format>R8G8B8</format>
+            </image>
+            <clip>
+              <near>0.02</near>
+              <far>10</far>
+            </clip>
+            <noise>
+              <type>gaussian</type>
+              <!-- Noise is sampled independently per pixel on each frame.
+                  That pixel's noise value is added to each of its color
+                    channels, which at that point lie in the range [0,1]. -->
+              <mean>0.0</mean>
+              <stddev>0.007</stddev>
+            </noise>
+          </camera>
+          <!-- <plugin name="depth_camera_controller" filename="libgazebo_ros_camera.so">
+            <camera_name>depth_camera</camera_name>
+            <frame_name>camera_depth_frame</frame_name>
+            <hack_baseline>0</hack_baseline>
+            <min_depth>0.001</min_depth>
+          </plugin> -->
+        </sensor>
       </link>
     <joint name="robot_camera_mount_joint" type="fixed">
